Commit message: Add CAD to URDF conversion playbook and related scripts
- Introduced a new documentation file `cad_to_urdf.md` detailing the process for converting CAD files to URDF, including prerequisites, steps, and common pitfalls.
- Created `convert_step_to_meshes.py` script to split the Epson T3-401S STEP assembly into individual STL meshes, applying necessary transformations and trimming for visual fidelity.
- Added `joint_trace.py` script for diagnosing arm stability by tracking joint positions and velocities during simulation.

File: assets/t3_401_simple_gripper/t3_401_simple_gripper.urdf (robot description, URDF)
Before this commit: robot t3_401_simple_gripper, 11 links, 10 joints
Links:
- link base_link: geometry collision cylinder length=0.50 radius=0.05; visual cylinder length=0.063 radius=0.05
- link link_1: geometry collision box size=0.225 0.06 0.040; visual mesh filename=meshes/link_1.stl scale=0.001 0.001 0.001
- link link_2: geometry collision box size=0.175 0.05 0.040; visual mesh filename=meshes/link_2.stl scale=0.001 0.001 0.001
- link link_3: geometry collision cylinder length=0.10 radius=0.012; visual mesh filename=meshes/link_3.stl scale=0.001 0.001 0.001

Commit message: Update T3-401 Tweezer assets and configurations for improved performance
- Updated STL mesh files for base_link, link_1, link_2, and link_3.
- Modified convert_step_to_meshes.py to reflect new part naming conventions.
- Adjusted TCP z-offset in pick_plant_out_of_vial.yaml for better alignment with the new tweezer design.
- Revised grasping and lifting parameters in pick_plant_out_of_vial.yaml and put_plant_back.yaml to accommodate the shorter tweezer.
- Enhanced success criteria and grasp-check parameters for more reliable operation.
- Added CLAUDE.md to document guidelines for sim-to-real fidelity and URDF/CAD handling.

File: assets/t3_401_simple_gripper/t3_401_simple_gripper.urdf (robot description, URDF)
Before this commit: robot t3_401_simple_gripper, 11 links, 10 joints
Links:
- link base_link: geometry collision cylinder length=0.50 radius=0.05; visual cylinder length=0.17 radius=0.10
Joints:
- joint joint_1: origin xyz=0 0 0.50 rpy=0 0 0 -> xyz=0 0 0.37 rpy=0 0 0
- joint joint_3: limit lower=0.0 upper=0.200 effort=120.0 velocity=1.0 -> lower=0.0 upper=0.150 effort=120.0 velocity=1.0; origin xyz=0.175 0 0 rpy=0 0 0 -> xyz=0.129 -0.023 0 rpy=0 0 0

Commit message: Refine T3-401 SCARA configurations and task parameters for improved performance and reliability

File: assets/t3_401_simple_gripper/t3_401_simple_gripper.urdf (robot description, URDF)
Before this commit: robot t3_401_simple_gripper, 11 links, 10 joints
Joints:
- joint joint_3: limit lower=0.0 upper=0.150 effort=120.0 velocity=1.0 -> lower=0.0 upper=0.200 effort=120.0 velocity=1.0; origin xyz=0.129 -0.023 0 rpy=0 0 0 -> xyz=0.175 0 0 rpy=0 0 0
